Commit message: Adjusting everything. Still issues with interference on overload of Ax-18s.

File: orchestration/packages/src/gummi_description/gummi.urdf (robot description, URDF)
Before this commit: robot gummi, 9 links, 8 joints
Links:
- link base_link: mass 1 -> None

Commit message: Ready for interaction test.

File: orchestration/packages/src/gummi_description/gummi.urdf (robot description, URDF)
Before this commit: robot gummi, 9 links, 8 joints
Joints:
- joint elbow: limit lower=-0.75 upper=0.85 effort=0 velocity=1.0 -> lower=-0.85 upper=0.85 effort=0 velocity=1.0
- joint shoulder_roll: limit lower=-0.2 upper=1.25 effort=0 velocity=1.0 -> lower=-0.55 upper=1.4 effort=0 velocity=1.0

Commit message: Not yet working, but ok in rviz.

File: orchestration/packages/src/gummi_description/gummi.urdf (robot description, URDF)
Before this commit: robot gummi, 9 links, 8 joints
Links:
- added link shoulder_intermediate; collision cylinder length=0.01 radius=0.065; visual cylinder length=0.01 radius=0.065
- added link shoulder_preroll; collision cylinder length=0.01 radius=0.065; visual cylinder length=0.01 radius=0.065
- link base_link: geometry collision cylinder length=0.01 radius=0.065; visual cylinder length=0.01 radius=0.065
- link coupling: geometry collision cylinder length=0.01 radius=0.02; visual cylinder length=0.01 radius=0.02
- link lowerarm: geometry collision cylinder length=0.11 radius=0.04; visual cylinder length=0.11 radius=0.04
- link lowerarm_preroll: geometry collision cylinder length=0.06 radius=0.03; visual cylinder length=0.06 radius=0.03
- link shoulder: geometry collision cylinder length=0.12 radius=0.06; visual cylinder length=0.12 radius=0.06
- link tool: geometry collision cylinder length=0.03 radius=0.04; visual cylinder length=0.03 radius=0.04
- link upperarm: geometry collision cylinder length=0.16 radius=0.04; visual cylinder length=0.16 radius=0.04
- link upperarm_preroll: geometry collision cylinder length=0.06 radius=0.03; visual cylinder length=0.06 radius=0.03
- link wrist: geometry collision cylinder length=0.04 radius=0.02; visual cylinder length=0.04 radius=0.02
Joints:
- added joint shoulder_fake: type fixed, parent shoulder_intermediate, child shoulder_preroll, origin xyz=0.0 0.0 0.0 rpy=0.0 0.0 1.57079, axis 0 0 1, limit lower=-0.52 upper=1.04 effort=0 velocity=1.0
- added joint shoulder_yaw: type revolute, parent base_link, child shoulder_intermediate, origin xyz=0.0 0.0 0.0 rpy=0.0 0.0 0.0, axis 0 0 1, limit lower=-0.52 upper=1.04 effort=0 velocity=1.0
- joint shoulder_roll: parent base_link -> shoulder_preroll

Commit message: Working 7DOF teleop, should now try weighting joints.

File: orchestration/packages/src/gummi_description/gummi.urdf (robot description, URDF)
Before this commit: robot gummi, 11 links, 10 joints
Links:
- removed link shoulder_intermediate
Joints:
- removed joint shoulder_fake
- joint shoulder_yaw: child shoulder_intermediate -> shoulder_preroll

Commit message: Found differences in naming of joints (todo: central), now ok pose control.

File: orchestration/packages/src/gummi_description/gummi.urdf (robot description, URDF)
Before this commit: robot gummi, 10 links, 9 joints
Joints:
- removed joint lowerarm_roll
- added joint forearm_roll: type revolute, parent lowerarm_preroll, child lowerarm, origin xyz=0.0 -0.079 0.0 rpy=1.57079 0.0 0.0, axis 0 0 1, limit lower=-2.7489 upper=2.7489 effort=0 velocity=1.0

Commit message: Reducing max angle of shoulder pitch, for now.
Former-commit-id: 51ec02b0c78f1b95fd418b547ff2ecc14c992b4e

File: orchestration/packages/src/gummi_description/gummi.urdf (robot description, URDF)
Before this commit: robot gummi, 10 links, 9 joints
Joints:
- joint shoulder_pitch: limit lower=0.0 upper=1.75 effort=0 velocity=1.0 -> lower=0.0 upper=1.1 effort=0 velocity=1.0

Commit message: Using full elbow range.
Former-commit-id: 006f8675377576dc44a0a4f4f0b6a69d6c9c37b5

File: orchestration/packages/src/gummi_description/gummi.urdf (robot description, URDF)
Before this commit: robot gummi, 10 links, 9 joints
Joints:
- joint elbow: limit lower=-0.85 upper=0.85 effort=0 velocity=1.0 -> lower=-0.85 upper=0.65 effort=0 velocity=1.0

Commit message: Better calibration (full range), now of full arm.
Former-commit-id: 9a31192def98458b2506cac7405faf2a6e310f39

File: orchestration/packages/src/gummi_description/gummi.urdf (robot description, URDF)
Before this commit: robot gummi, 10 links, 9 joints
Joints:
- joint wrist_pitch: limit lower=-1.0 upper=1.0 effort=0 velocity=1.0 -> lower=-0.9 upper=0.6 effort=0 velocity=1.0

Commit message: Lower arm rotated 90 degrees inwards.
Former-commit-id: bb80be88d40fab6b68fe0df4a31f74296afaf685

File: orchestration/packages/src/gummi_description/gummi.urdf (robot description, URDF)
Before this commit: robot gummi, 10 links, 9 joints
Joints:
- joint wrist_pitch: origin xyz=0.0 0.0 0.15 rpy=-1.57079 0.0 0.0 -> xyz=0.0 0.0 0.15 rpy= 0.0 1.57079 0.0

Commit message: Reduced pull on wrist to avoid overheating.
Former-commit-id: 688263f08462cd5b6ca8de98d9b2373138890c05

File: orchestration/packages/src/gummi_description/gummi.urdf (robot description, URDF)
Before this commit: robot gummi, 10 links, 9 joints
Joints:
- joint wrist_pitch: limit lower=-0.9 upper=0.6 effort=0 velocity=1.0 -> lower=-0.75 upper=0.5 effort=0 velocity=1.0

Commit message: Better URDF, 15 deg condition for cocontraction, and full arm test ok.
Former-commit-id: ad5dc139e12b09d9358f66f81361f8bac21b30ed

File: orchestration/packages/src/gummi_description/gummi.urdf (robot description, URDF)
Before this commit: robot gummi, 10 links, 9 joints
Joints:
- joint wrist_to_coupling: origin xyz=0.0 -0.0281 0.0 rpy=0.0 0.0 -1.57079 -> xyz=-0.0281 0.0 0.0 rpy=0.0 0.0 3.14159

Commit message: Wider range for shoulder pitch.
Former-commit-id: e6b6f4c1463707bfade464a0ec11ab9e255b55dd

File: orchestration/packages/src/gummi_description/gummi.urdf (robot description, URDF)
Before this commit: robot gummi, 10 links, 9 joints
Joints:
- joint shoulder_pitch: limit lower=0.0 upper=1.1 effort=0 velocity=1.0 -> lower=-0.1 upper=1.1 effort=0 velocity=1.0

Commit message: Need to go over mapping for forward models.
Former-commit-id: 2b90ad457dbf5ade102995b9c92a7aea94f12b7b

File: orchestration/packages/src/gummi_description/gummi.urdf (robot description, URDF)
Before this commit: robot gummi, 10 links, 9 joints
Joints:
- joint shoulder_pitch: limit lower=-0.1 upper=1.1 effort=0 velocity=1.0 -> lower=-0.15 upper=1.1 effort=0 velocity=1.0

Commit message: Rotated wrist ala ghost for teleop.

File: orchestration/packages/src/gummi_description/gummi.urdf (robot description, URDF)
Before this commit: robot gummi, 10 links, 9 joints
Joints:
- joint wrist_pitch: axis 0 0 1 -> 0 1 0; limit lower=-0.75 upper=0.5 effort=0 velocity=1.0 -> lower=-0.75 upper=0.75 effort=0 velocity=1.0

Commit message: almost ready for testing but arm not behaving well

File: orchestration/packages/src/gummi_description/gummi.urdf (robot description, URDF)
Before this commit: robot gummi, 10 links, 9 joints
Joints:
- joint elbow: limit lower=-0.85 upper=0.65 effort=0 velocity=1.0 -> lower=-0.85 upper=0.47 effort=0 velocity=1.0
- joint shoulder_roll: limit lower=-0.55 upper=1.4 effort=0 velocity=1.0 -> lower=-1.4 upper=2.4 effort=0 velocity=1.0
- joint wrist_pitch: limit lower=-0.75 upper=0.75 effort=0 velocity=1.0 -> lower=-0.75 upper=0.5 effort=0 velocity=1.0
